File: WashingLineMonitor-P0001.kicad_pcb (KiCad board)
At the start: 2 copper layers, 58.5 x 41.5 mm, 51 parts, among them J1 Conn_01x02_Socket, J3 Conn_02x03_Odd_Even, U1 ESP32-S2-SOLO-2-N4, U2 TLV2371DBV, U4 AP2112K-3.3, U6 BQ51050BRHL

Commit message: commit of local files before designing next version
Other:
- board text added: "HoratioPistachio WashingLineMonitor-P0001_AB"
- board text removed: "HoratioPistachio WashingLineMonitor-P0001_AA"
Changed lines of the file:
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@@
 		(end 46.188458 26.930276)
 		(stroke
-			(width 0)
+			(width 0.1)
 			(type solid)
 		)
@@
 		(layer "Edge.Cuts")
 	)
-	(gr_text "HoratioPistachio\nWashingLineMonitor-P0001_AA"
+	(gr_text "HoratioPistachio\nWashingLineMonitor-P0001_AB"
 		(at 39.5 21 0)
 		(layer "F.SilkS")

Commit message: laid out pcb
Parts:
- removed D1: MBR0530, Diode_SMD:D_SOD-123
- removed R3, R4: 500k, Resistor_SMD:R_0805_2012Metric_Pad1.20x1.40mm_HandSolder
- removed U4: AP2112K-3.3, Package_TO_SOT_SMD:SOT-23-5
- added C24: 100nF, Capacitor_SMD:C_0805_2012Metric_Pad1.18x1.45mm_HandSolder, F.Cu at (92.5, 38.9)
- added C25: 22uF, Capacitor_SMD:C_0805_2012Metric_Pad1.18x1.45mm_HandSolder, F.Cu at (71.5, 39.4)
- added D3: LED, LED_SMD:LED_0805_2012Metric_Pad1.15x1.40mm_HandSolder, F.Cu at (93.5, 33.5)
- added J2: S1711-46R, Hydro_footprints:HARWIN_S1711-46R, F.Cu at (62.5, 50.0)
- added JP1: Jumper_2_Bridged, Jumper:SolderJumper-2_P1.3mm_Bridged_RoundedPad1.0x1.5mm, F.Cu at (56.5, 36.9)
- added NTC1: TestPoint, TestPoint:TestPoint_Pad_D1.0mm, F.Cu at (62.0, 21.2)
- added Q1: PJA3401A_R1_00001, Package_TO_SOT_SMD:SOT-23, F.Cu at (60.4, 37.9)
- added Q3: Q_Dual_NMOS_PMOS_G1S2G2D2S1D1, Package_SO:TSOP-6_1.65x3.05mm_P0.95mm, F.Cu at (47.5, 39.3)
- added R12: 2.4k, Resistor_SMD:R_0805_2012Metric_Pad1.20x1.40mm_HandSolder, F.Cu at (91.0, 33.5)
- added R13: 10k, Resistor_SMD:R_0805_2012Metric_Pad1.20x1.40mm_HandSolder, F.Cu at (85.0, 38.4)
- added R14: 10k, Resistor_SMD:R_0805_2012Metric_Pad1.20x1.40mm_HandSolder, F.Cu at (87.5, 34.0)
- added R15: 10k, Resistor_SMD:R_0805_2012Metric_Pad1.20x1.40mm_HandSolder, F.Cu at (56.5, 40.4)
- added R16: 500k, Resistor_SMD:R_0805_2012Metric_Pad1.20x1.40mm_HandSolder, F.Cu at (61.0, 40.9)
- added R17: 10k, Resistor_SMD:R_0805_2012Metric_Pad1.20x1.40mm_HandSolder, F.Cu at (46.0, 43.5)
- added R18: 10k, Resistor_SMD:R_0805_2012Metric_Pad1.20x1.40mm_HandSolder, F.Cu at (48.5, 43.5)
- added R19: 10k, Resistor_SMD:R_0805_2012Metric_Pad1.20x1.40mm_HandSolder, F.Cu at (51.0, 43.5)
- added R20: 500k, Resistor_SMD:R_0805_2012Metric_Pad1.20x1.40mm_HandSolder, F.Cu at (47.5, 36.0)
- added SW1: A6TN-1104, Button_Switch_THT:SW_DIP_SPSTx01_Slide_6.7x4.1mm_W7.62mm_P2.54mm_LowProfile, F.Cu at (69.0, 33.5)
- added T2: TestPoint, TestPoint:TestPoint_Pad_D1.0mm, B.Cu at (91.2, 37.0)
- added TH1: Thermistor_NTC, Resistor_SMD:R_0402_1005Metric_Pad0.72x0.64mm_HandSolder, B.Cu at (60.5, 25.0)
- added U3: ESP32-C6-MINI-1, RF_Module:ESP32-C6-MINI-1, F.Cu at (87.1, 25.1)
- added U5: TLV75533PDBV, Package_TO_SOT_SMD:SOT-23-5, F.Cu at (65.3, 38.9)
- added Vbatt2: TestPoint, TestPoint:TestPoint_Pad_D1.0mm, F.Cu at (53.0, 40.0)
- BT3: footprint Connector_Wire:SolderWire-0.1sqmm_1x02_P3.6mm_D0.4mm_OD1mm_Relief -> Connector_JST:JST_SH_SM02B-SRSS-TB_1x02-1MP_P1.00mm_Horizontal; moved to F.Cu
- D2: value BZX84C3V3-7-F -> BZX84C5V1-TP
- J1: value Conn_01x02_Socket -> S1711-46R; footprint Connector_Wire:SolderWire-0.1sqmm_1x02_P3.6mm_D0.4mm_OD1mm_Relief -> Hydro_footprints:HARWIN_S1711-46R
- L1: footprint Connector_Wire:SolderWire-0.1sqmm_1x02_P3.6mm_D0.4mm_OD1mm_Relief -> Connector_JST:JST_SH_SM02B-SRSS-TB_1x02-1MP_P1.00mm_Horizontal
- R10: value 10k -> 500k
- U1: value ESP32-S2-SOLO-2-N4 -> HDC2080; footprint Hydro_footprints:ESP32-S2-SOLO-N4 -> Sensor_Humidity:Texas_S-PWSON-N6-HDC2080
- moved C20 22.3 mm to (67.5, 36.0), turned to 180 degrees
- moved R10 19.0 mm to (51.0, 39.0)
- moved C18 15.4 mm to (47.0, 32.5), turned to -90 degrees
- moved C19 14.3 mm to (78.5, 32.0), turned to 0 degrees
- moved Vsense1 14.1 mm to (74.0, 36.0), turned to -90 degrees
- moved C17 14.0 mm to (50.0, 32.5), turned to -90 degrees
- moved C22 13.9 mm to (53.5, 43.5), turned to 90 degrees
- moved SenseOut1 13.8 mm to (78.0, 30.0), turned to -90 degrees
- moved C21 13.7 mm to (69.0, 39.4), turned to 90 degrees
- moved R1 13.5 mm to (75.0, 38.5), turned to 0 degrees
- moved C3 13.3 mm to (48.5, 29.2)
- moved R11 13.2 mm to (80.5, 44.0), turned to 90 degrees
- moved BattMeas1 13.1 mm to (56.5, 44.5), turned to -90 degrees
- moved C23 13.1 mm to (78.0, 44.0), turned to -90 degrees
- moved C4 12.8 mm to (48.4, 26.7)
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Connections:
- R10 pad 1: GND -> Net-(Q3A-G)
- R10 pad 2: NTC_BATT -> Vbatt
- U1 pad 1: GND -> SDA
- U1 pad 2: 3V3 -> GND
- U1 pad 3: ESP_EN -> GND
- U1 pad 4: unconnected-(U1-IO4-Pad4) -> HDC_INT
- U1 pad 5: unconnected-(U1-IO5-Pad5) -> HDC_POWER
- U1 pad 6: unconnected-(U1-IO6-Pad6) -> SCL
- Vbatt1 pad 1: Vbatt -> Net-(Q3A-S)
Routing:
- net MEAS_BATT: track 0.00 -> 63.0 mm, vias 0 -> 4
- net CHARGE_STATUS: track 16.3 -> 46.9 mm, vias 0 -> 2
- net HDC_POWER: track 0.00 -> 29.9 mm
- net QI_EN2: track 10.7 -> 39.3 mm, vias 0 -> 2
- net 3V3: track 84.4 -> 56.8 mm
- net Net-(U5-EN): track 0.00 -> 22.0 mm
- net Battery_Voltage: track 24.9 -> 46.1 mm
- net Vbatt: track 9.97 -> 30.0 mm
- net Net-(U6-AC2): track 8.93 -> 26.1 mm
- net ESP_BOOT: track 10.0 -> 25.2 mm
- net Net-(U6-AC1): track 11.7 -> 25.8 mm
- net HDC_INT: track 0.00 -> 13.1 mm, vias 0 -> 2
- net ESP_EN: track 39.6 -> 28.4 mm, vias 2 -> 4
- net SDA: track 0.00 -> 9.89 mm
- net SCL: track 0.00 -> 9.33 mm
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- removed copper zone on F.Cu, net Net-(C3-Pad1)
- removed copper zone on F.Cu, net Net-(U6-AC1)
- removed copper zone on F.Cu, net Net-(U6-AC2)
Other:
- outline, holes or cut-outs redrawn
- board text added: "HoratioPistachio WashingLineMonitor-P0001_AC"
- board text removed: "HoratioPistachio WashingLineMonitor-P0001_AB"

Commit message: Near complete AC
Parts:
- moved TP7 6.00 mm to (62.5, 44.5)
- moved TP5 5.77 mm to (54.8, 34.5)
- moved R20 3.50 mm to (51.0, 36.0)
- moved L1 2.88 mm to (44.9, 27.0)
- moved BT3 2.50 mm to (44.5, 35.0)
- moved C22 2.50 mm to (56.0, 43.5)
- moved Q3 2.50 mm to (50.0, 39.3)
- moved R10 2.50 mm to (53.5, 39.0)
- moved R17 2.50 mm to (48.5, 43.5)
- moved R18 2.50 mm to (51.0, 43.5)
- moved R19 2.50 mm to (53.5, 43.5)
- moved TP6 2.50 mm to (47.0, 39.5)
- moved J2 2.32 mm to (62.2, 52.3)
- moved J1 2.31 mm to (70.3, 52.3)
- moved C10 2.00 mm to (58.2, 20.5)
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- renumbered Vsense1 to TP1, NTC1 to TP10, SenseOut1 to TP2, GND1 to TP3, T2 to TP4, Vbatt2 to TP5, Vbatt1 to TP6, BattMeas1 to TP7, 3V3 to TP8, AD-EN1 to TP9
Connections:
- Q1 pad 1: Net-(JP1-B) -> Net-(Q1-G)
- Q1 pad 2: Net-(Q1-G) -> Net-(Q1-S)
- Q1 pad 3: Net-(Q1-S) -> Net-(JP1-B)
Routing:
- net MEAS_BATT: track 63.0 -> 58.9 mm
- net GND: track 14.0 -> 16.4 mm, vias 51 -> 64
- net Vbatt: track 30.0 -> 27.7 mm
- net QI_EN2: track 39.3 -> 37.3 mm
- net ESP_EN: track 28.4 -> 26.6 mm
- net Net-(U6-AC2): track 26.1 -> 24.3 mm
- net Net-(JP1-B): track 2.35 -> 3.55 mm
- net RXD0: track 24.1 -> 23.0 mm
- net Net-(D3-A): track 3.55 -> 2.51 mm
- net Net-(C3-Pad1): track 8.77 -> 7.89 mm
- net Net-(Q1-G): track 2.64 -> 3.36 mm
- net CHARGE_STATUS: track 46.9 -> 46.2 mm
Other:
- board size 58.5 x 41.5 mm -> 58.5 x 43.5 mm

Commit message: Minor pre release changes
Parts:
- added FID1: Fiducial, Fiducial:Fiducial_0.5mm_Mask1mm, F.Cu at (119.5, 105.5)
- added FID2: Fiducial, Fiducial:Fiducial_0.5mm_Mask1mm, F.Cu at (120.5, 75.0)
- added FID3: Fiducial, Fiducial:Fiducial_0.5mm_Mask1mm, F.Cu at (162.5, 106.0)
- moved C4 98.8 mm to (130.4, 84.7)
- moved J1 98.8 mm to (150.3, 110.3)
- moved Q3 98.8 mm to (130.1, 97.3)
- moved BT3 98.8 mm to (124.5, 93.0)
- moved C1 98.8 mm to (157.0, 83.0)
- moved C11 98.8 mm to (135.0, 89.2)
- moved C12 98.8 mm to (141.0, 91.5)
- moved C13 98.8 mm to (138.0, 91.5)
- moved C16 98.8 mm to (133.0, 74.2)
- moved C17 98.8 mm to (132.0, 90.5)
- moved C18 98.8 mm to (129.0, 90.5)
- moved C19 98.8 mm to (158.5, 90.0)
- moved C2 98.8 mm to (157.0, 80.5)
- moved C20 98.8 mm to (147.5, 94.0)
- moved C21 98.8 mm to (149.0, 97.4)
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Routing:
- net GND: vias 64 -> 65
Other:
- board text added: "+-"
- board text added: "GND"
