File: qi_wireless_power.kicad_sch (KiCad schematic)
At the start: 24 parts, among them U3 NTJD4152PT1G, U6 BQ51050BRHL

Commit message: Completed first iteration and reviews
Parts:
- removed D1: MBR0530, Diode_SMD:D_SOD-123, symbol Diode:MBR0530
- removed U3: NTJD4152PT1G, Package_TO_SOT_SMD:SOT-363_SC-70-6_Handsoldering, symbol Hydro_symbols:NTJD4152PT1G
- added AD-EN1: TestPoint, TestPoint:TestPoint_Pad_D1.0mm, symbol Connector:TestPoint
- added C3: 4.7uF, Capacitor_SMD:C_0805_2012Metric_Pad1.18x1.45mm_HandSolder, symbol Device:C
- BT3: footprint (none) -> Connector_Wire:SolderWire-0.1sqmm_1x02_P3.6mm_D0.4mm_OD1mm_Relief; Supplier (none) -> Core Electronics; Supplier Part Number (none) -> CE04377
- C10, C13: footprint (none) -> Capacitor_SMD:C_0805_2012Metric_Pad1.18x1.45mm_HandSolder; Supplier (none) -> Digikey; Supplier Part Number (none) -> 1276-2488-1-ND
- C11, C8: footprint (none) -> Capacitor_SMD:C_0805_2012Metric_Pad1.18x1.45mm_HandSolder; Supplier (none) -> Digikey; Supplier Part Number (none) -> 1276-1015-1-ND
- C12, C9: footprint (none) -> Capacitor_SMD:C_0805_2012Metric_Pad1.18x1.45mm_HandSolder; Supplier (none) -> Digikey; Supplier Part Number (none) -> 1276-6480-1-ND
- C14, C15: footprint (none) -> Capacitor_SMD:C_0805_2012Metric_Pad1.18x1.45mm_HandSolder; Supplier (none) -> Digikey; Supplier Part Number (none) -> 1276-1096-1-ND
- C16, C17: footprint (none) -> Capacitor_SMD:C_0805_2012Metric_Pad1.18x1.45mm_HandSolder; Supplier (none) -> Digikey; Supplier Part Number (none) -> 1276-1003-1-ND
- C18: footprint (none) -> Capacitor_SMD:C_0805_2012Metric_Pad1.18x1.45mm_HandSolder; Supplier (none) -> Digikey; Supplier Part Number (none) -> 1276-1029-1-ND
- C4: value 1uF -> 4.7uF; footprint (none) -> Capacitor_SMD:C_0805_2012Metric_Pad1.18x1.45mm_HandSolder; Supplier (none) -> Digikey; Supplier Part Number (none) -> 1276-1244-1-ND
- C5: value 18uF -> 10uF; footprint (none) -> Capacitor_SMD:C_0805_2012Metric_Pad1.18x1.45mm_HandSolder; Supplier (none) -> Digikey; Supplier Part Number (none) -> 1276-1096-1-ND
- C6, C7: footprint (none) -> Capacitor_SMD:C_0805_2012Metric_Pad1.18x1.45mm_HandSolder; Supplier (none) -> Digikey; Supplier Part Number (none) -> 1276-2425-1-ND
- L1: footprint (none) -> Connector_Wire:SolderWire-0.1sqmm_1x02_P3.6mm_D0.4mm_OD1mm_Relief; Supplier (none) -> Digikey; Supplier Part Number (none) -> 445-16091-ND
- R10: value 10kR -> 10k; footprint (none) -> Resistor_SMD:R_0805_2012Metric_Pad1.20x1.40mm_HandSolder; Supplier (none) -> Digikey; Supplier Part Number (none) -> P10KACT-ND
- R7: value 430R -> 430; footprint (none) -> Resistor_SMD:R_0805_2012Metric_Pad1.20x1.40mm_HandSolder; Supplier (none) -> Digikey; Supplier Part Number (none) -> P430DACT-ND
- R8: value 2.4kR -> 2.4k; footprint (none) -> Resistor_SMD:R_0805_2012Metric_Pad1.20x1.40mm_HandSolder; Supplier (none) -> Digikey; Supplier Part Number (none) -> P2.4KDACT-ND
- R9: value 20kR -> 20k; footprint (none) -> Resistor_SMD:R_0805_2012Metric_Pad1.20x1.40mm_HandSolder; Supplier (none) -> Digikey; Supplier Part Number (none) -> P20KACT-ND
- U6: Supplier (none) -> Digikey; Supplier Part Number (none) -> 296-BQ51050BRHLRCT-ND
Connections:
- net Vusb is gone; now on net GND: U6.9 (AD)
- net NTC_BATT: now reaches R10.2, U6.13 (TS/CTRL)
- net at C11.2, C12.2, C13.2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: now also C3.2
- net at U6.8 (~{AD-EN}): now also AD-EN1.1
- net at C4.1, C5.1, L1.2: now also C3.1
Other:
- company: (none) -> Horatio Pistachio
- title: (none) -> WashingLineMonitor-P0001
- moved on the sheet: C4

Commit message: commit of local files before designing next version
Parts:
- L1: JLC_Part_Number (none) -> C5331042
- U6: JLC_Part_Number (none) -> C2650144
Changed lines of the file:
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@@
+			)
+		)
+		(property "JLC_Part_Number" "C2650144"
+			(at 180.34 81.28 0)
+			(effects
+				(font
+					(size 1.27 1.27)
+				)
+				(hide yes)
 			)
 		)
@@
 			)
 		)
+		(property "JLC_Part_Number" ""
+			(at 121.92 90.17 0)
+			(effects
+				(font
+					(size 1.27 1.27)
+				)
+				(hide yes)
+			)
+		)
 		(pin "2"
 		)
@@
 			)
 		)
+		(property "JLC_Part_Number" "C5331042"
+			(at 91.44 83.82 0)
+			(effects
+				(font
+					(size 1.27 1.27)
+				)
+				(hide yes)
+			)
+		)
 		(pin "1"
 		)
@@
 			)
 		)
+		(property "JLC_Part_Number" ""
+			(at 160.02 60.96 0)
+			(effects
+				(font
+					(size 1.27 1.27)
+				)
+				(hide yes)
+			)
+		)
 		(pin "1"
 		)
@@
 			)
 		)
+		(property "JLC_Part_Number" ""
+			(at 135.89 132.08 90)
+			(effects
+				(font
+					(size 1.27 1.27)
+				)
+				(hide yes)
+			)
+		)
 		(pin "2"
 		)
@@
 			)
 		)
+		(property "JLC_Part_Number" ""
+			(at 121.92 78.74 0)
+			(effects
+				(font
+					(size 1.27 1.27)
+				)
+				(hide yes)
+			)
+		)
 		(pin "2"
 		)
@@
 			)
 		)
+		(property "JLC_Part_Number" ""
+			(at 134.62 24.13 90)
+			(effects
+				(font
+					(size 1.27 1.27)
+				)
+				(hide yes)
+			)
+		)
 		(pin "2"
 		)
@@
 			)
 		)
+		(property "JLC_Part_Number" ""
+			(at 267.97 110.49 0)
+			(effects
+				(font
+					(size 1.27 1.27)
+				)
+				(hide yes)
+			)
+		)
 		(pin "2"
 		)
@@
 			)
 		)
+		(property "JLC_Part_Number" ""
+			(at 109.22 72.39 90)
+			(effects
+				(font
+					(size 1.27 1.27)
+				)
+				(hide yes)
+			)
+		)
 		(pin "2"
 		)
@@
 			)
 		)
+		(property "JLC_Part_Number" ""
+			(at 228.6 68.58 0)
+			(effects
+				(font
+					(size 1.27 1.27)
+				)
+				(hide yes)
+			)
+		)
 		(pin "2"
 		)
@@
 			)
 		)
+		(property "JLC_Part_Number" ""
+			(at 245.11 68.58 0)
+			(effects
+				(font
+					(size 1.27 1.27)
+				)
+				(hide yes)
+			)
+		)
 		(pin "2"
 		)
@@
 			)
 		)
+		(property "JLC_Part_Number" ""
+			(at 219.71 87.63 0)
+			(effects
+				(font
+					(size 1.27 1.27)
+				)
+				(hide yes)
+			)
+		)
 		(pin "1"
 		)
@@
 			)
 		)
+		(property "JLC_Part_Number" ""
+			(at 134.62 38.1 90)
+			(effects
+				(font
+					(size 1.27 1.27)
+				)
+				(hide yes)
+			)
+		)
 		(pin "2"
 		)
@@
 			)
 		)
+		(property "JLC_Part_Number" ""
+			(at 245.11 110.49 0)
+			(effects
+				(font
+					(size 1.27 1.27)
+				)
+				(hide yes)
+			)
+		)
 		(pin "2"
 		)
@@
 			)
 		)
+		(property "JLC_Part_Number" ""
+			(at 135.89 119.38 90)
+			(effects
+				(font
+					(size 1.27 1.27)
+				)
+				(hide yes)
+			)
+		)
 		(pin "2"
 		)
@@
 			)
 		)
+		(property "JLC_Part_Number" ""
+			(at 134.62 53.34 90)
+			(effects
+				(font
+					(size 1.27 1.27)
+				)
+				(hide yes)
+			)
+		)
 		(pin "2"
 		)
@@
 			)
 		)
+		(property "JLC_Part_Number" ""
+			(at 196.85 105.41 0)
+			(effects
+				(font
+					(size 1.27 1.27)
+				)
+				(hide yes)
+			)
+		)
 		(pin "1"
 		)
@@
 			)
 		)
+		(property "JLC_Part_Number" ""
+			(at 109.22 45.72 90)
+			(effects
+				(font
+					(size 1.27 1.27)
+				)
+				(hide yes)
+			)
+		)
 		(pin "2"
 		)
@@
 			)
 		)
+		(property "JLC_Part_Number" ""
+			(at 264.16 71.12 0)
+			(effects
+				(font
+					(size 1.27 1.27)
+				)
+				(hide yes)
+			)
+		)
 		(pin "1"
 		)
@@
 			)
 		)
+		(property "JLC_Part_Number" ""
+			(at 231.14 91.44 90)
+			(effects
+				(font
+					(size 1.27 1.27)
+				)
+				(hide yes)
+			)
+		)
 		(pin "1"
 		)
@@
 			)
 		)
+		(property "JLC_Part_Number" ""
+			(at 135.89 106.68 90)
+			(effects
+				(font
+					(size 1.27 1.27)
+				)
+				(hide yes)
+			)
+		)
 		(pin "2"
 		)
@@
 			)
 		)
+		(property "JLC_Part_Number" ""
+			(at 109.22 59.69 90)
+			(effects
+				(font
+					(size 1.27 1.27)
+				)
+				(hide yes)
+			)
+		)
 		(pin "2"
 		)
@@
 			)
 		)
+		(property "JLC_Part_Number" ""
+			(at 256.54 110.49 0)
+			(effects
+				(font
+					(size 1.27 1.27)
+				)
+				(hide yes)
+			)
+		)
 		(pin "2"
 		)
@@
 			(at 207.01 105.41 0)
 			(effects
+				(font
+					(size 1.27 1.27)
+				)
+				(hide yes)
+			)
+		)
+		(property "JLC_Part_Number" ""
+			(at 207.01 105.41 0)
+			(effects

Commit message: updated schematic from review
Parts:
- removed R10: 10k, Resistor_SMD:R_0805_2012Metric_Pad1.20x1.40mm_HandSolder, symbol Device:R
- added NTC1: TestPoint, TestPoint:TestPoint_Pad_D1.0mm, symbol Connector:TestPoint
- added TH1: Thermistor_NTC, Resistor_SMD:R_0402_1005Metric_Pad0.72x0.64mm_HandSolder, symbol Device:Thermistor_NTC
Connections:
- net GND: now also TH1.2
- net NTC_BATT: now also NTC1.1, TH1.1

Commit message: laid out pcb
Parts:
- BT3, L1: footprint Connector_Wire:SolderWire-0.1sqmm_1x02_P3.6mm_D0.4mm_OD1mm_Relief -> Connector_JST:JST_SH_SM02B-SRSS-TB_1x02-1MP_P1.00mm_Horizontal
Changed lines of the file:
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@@
 			)
 		)
-		(property "Footprint" "Connector_Wire:SolderWire-0.1sqmm_1x02_P3.6mm_D0.4mm_OD1mm_Relief"
+		(property "Footprint" "Connector_JST:JST_SH_SM02B-SRSS-TB_1x02-1MP_P1.00mm_Horizontal"
 			(at 91.44 83.82 0)
 			(hide yes)
@@
 			)
 		)
-		(property "Footprint" "Connector_Wire:SolderWire-0.1sqmm_1x02_P3.6mm_D0.4mm_OD1mm_Relief"
+		(property "Footprint" "Connector_JST:JST_SH_SM02B-SRSS-TB_1x02-1MP_P1.00mm_Horizontal"
 			(at 264.16 69.596 90)
 			(hide yes)

Commit message: Near complete AC
Parts:
- BT3: Description_1 (none) -> CE04377; Supplier Part Number CE04377 -> 455-SM02B-SRSS-TBCT-ND
- L1: Availability (none) -> 445-16091-ND; Supplier Part Number 445-16091-ND -> 455-SM02B-SRSS-TBCT-ND
- renumbered NTC1 to TP10, AD-EN1 to TP9
Changed lines of the file:
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@@
 		(dnp no)
 		(fields_autoplaced yes)
-		(property "Reference" "NTC1"
+		(property "Reference" "TP10"
 			(at 201.93 71.6279 0)
 			(show_name no)
@@
 			(project "WashingLineMonitor-P0001"
 				(path "/09468f75-1295-4aed-9d66-1cbb46f6d9f7/fe242c69-4638-4ad9-952b-9c215da932fb/2f2216a8-e089-410a-a3dd-67c68912bcc4"
-					(reference "NTC1")
+					(reference "TP10")
 					(unit 1)
 				)
@@
 			)
 		)
-		(property "Supplier Part Number" "445-16091-ND"
+		(property "Supplier Part Number" "455-SM02B-SRSS-TBCT-ND"
 			(at 91.44 83.82 0)
 			(hide yes)
@@
 			)
 		)
-		(property "Availability" ""
+		(property "Availability" "445-16091-ND"
 			(at 91.44 83.82 0)
 			(hide yes)
@@
 		(dnp no)
 		(fields_autoplaced yes)
-		(property "Reference" "AD-EN1"
+		(property "Reference" "TP9"
 			(at 162.56 56.3879 0)
 			(show_name no)
@@
 			(project "WashingLineMonitor-P0001"
 				(path "/09468f75-1295-4aed-9d66-1cbb46f6d9f7/fe242c69-4638-4ad9-952b-9c215da932fb/2f2216a8-e089-410a-a3dd-67c68912bcc4"
-					(reference "AD-EN1")
+					(reference "TP9")
 					(unit 1)
 				)
@@
 			)
 		)
-		(property "Supplier Part Number" "CE04377"
+		(property "Supplier Part Number" "455-SM02B-SRSS-TBCT-ND"
 			(at 264.16 71.12 0)
 			(hide yes)
@@
 			)
 		)
-		(property "Description_1" ""
+		(property "Description_1" "CE04377"
 			(at 264.16 71.12 0)
 			(hide yes)

Commit message: Minor pre release changes
Parts:
- TP10, TP9: now left out of the parts list
Changed lines of the file:
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@@
 	(title_block
 		(title "WashingLineMonitor-P0001")
-		(date "2025-09-14")
-		(rev "AB")
+		(date "2026-06-06")
+		(rev "AC")
 		(company "Horatio Pistachio")
 	)
@@
 		(body_style 1)
 		(exclude_from_sim no)
-		(in_bom yes)
+		(in_bom no)
 		(on_board yes)
 		(in_pos_files yes)
@@
 		(body_style 1)
 		(exclude_from_sim no)
-		(in_bom yes)
+		(in_bom no)
 		(on_board yes)
 		(in_pos_files yes)
